File: capacitive-touch/capacitive-touch-demo.sch (KiCad schematic (older format))
At the start: 21 parts, among them J1 Conn_01x05_Male, J2 AVR-ISP-6, Q1 BS170, U1 ATmega328P-PU, Y1 16MHz

Commit message: Rerutet og oppdaterte fotavtrykk på pcb til kapacativ touch
Parts:
- removed U1: ATmega328P-PU, Package_DIP:DIP-28_W7.62mm_LongPads, symbol MCU_Microchip_ATmega:ATmega328P-PU
- added C12: 100pF, Capacitor_SMD:C_1206_3216Metric_Pad1.42x1.75mm_HandSolder, symbol Device:C
- added C13: capacitive-pad, pads-cap-lib:capacitive-pad-small, symbol capacitive-pad:capacitive-pad
- added R6: 1M, Resistor_SMD:R_1206_3216Metric_Pad1.42x1.75mm_HandSolder, symbol Device:R
- added U1: ATmega168-20AU, Package_QFP:TQFP-32_7x7mm_P0.8mm, symbol MCU_Microchip_ATmega:ATmega168-20AU
Connections:
- net GND: now also C12.2, U1.21 (GND), U1.3 (GND), U1.5 (GND)
- net MISO: now also U1.16 (PB4)
- net MOSI: now also U1.15 (PB3)
- net RPin: now also U1.29 (~RESET~/PC6)
- net SCK: now also U1.17 (PB5)
- net SCL: now also J1.4 (Pin_4), U1.28 (PC5); no longer J1.3 (Pin_3)
- net SDA: now also J1.3 (Pin_3), U1.27 (PC4); no longer J1.4 (Pin_4)
- net VCC: now also U1.4 (VCC), U1.6 (VCC)
- net clk1: now also U1.7 (XTAL1/PB6)
- net clk2: now also U1.8 (XTAL2/PB7)
- net at C7.1, C8.1 (Pad), R4.2: now also U1.1 (PD3)
- net at R5.1: now also U1.10 (PD6)
- net at C10.1 (Pad), C9.1, R5.2: now also U1.9 (PD5)
- net at C3.1, C4.1 (Pad), R2.2: now also U1.30 (PD0)
- net at R2.1: now also U1.31 (PD1)
- net at R3.1: now also U1.25 (PC2)
- net at C5.1, C6.1 (Pad), R3.2: now also U1.26 (PC3)
- net at R4.1: now also U1.2 (PD4)
- new net: C12.1, C13.1 (Pad), R6.2, U1.11 (PD7)
- new net: R6.1, U1.12 (PB0)
Changed lines of the file:
@@
-	1    0    0    -1
-$EndComp
-$Comp
-L MCU_Microchip_ATmega:ATmega328P-PU U1
-U 1 1 5C0D6589
-P 4800 2550
-F 0 "U1" H 4159 2596 50  0000 R CNN
-F 1 "ATmega328P-PU" H 4159 2505 50  0000 R CNN
-F 2 "Package_DIP:DIP-28_W7.62mm_LongPads" H 4800 2550 50  0001 C CIN
-F 3 "http://ww1.microchip.com/downloads/en/DeviceDoc/ATmega328_P%20AVR%20MCU%20with%20picoPower%20Technology%20Data%20Sheet%2040001984A.pdf" H 4800 2550 50  0001 C CNN
-	1    4800 2550
 	1    0    0    -1
 $EndComp
@@
 Wire Wire Line
 	2250 2350 2150 2350
+Text Label 2400 2150 2    50   ~ 0
+SDA
 Text Label 2400 2250 2    50   ~ 0
-SDA
-Text Label 2400 2150 2    50   ~ 0
 SCL
 Wire Wire Line
@@
 Wire Wire Line
 	5400 2750 5650 2750
-$Comp
-L capacitive-pad:capacitive-pad C4
-U 1 1 5C6F29A5
-P 7450 1600
-F 0 "C4" H 7677 1646 50  0000 L CNN
-F 1 "capacitive-pad" H 7677 1555 50  0000 L CNN
-F 2 "pads-cap-lib:capacitive-pad" H 7450 1600 50  0001 C CNN
-F 3 "" H 7450 1600 50  0001 C CNN
-	1    7450 1600
-	1    0    0    -1
-$EndComp
 Wire Wire Line
 	7150 1150 7150 1600
@@
 	7300 2250 7150 2250
 Connection ~ 7150 2250
-$Comp
-L capacitive-pad:capacitive-pad C6
-U 1 1 5C6F49E6
-P 7450 2700
-F 0 "C6" H 7677 2746 50  0000 L CNN
-F 1 "capacitive-pad" H 7677 2655 50  0000 L CNN
-F 2 "pads-cap-lib:capacitive-pad" H 7450 2700 50  0001 C CNN
-F 3 "" H 7450 2700 50  0001 C CNN
-	1    7450 2700
-	1    0    0    -1
-$EndComp
 Wire Wire Line
 	7150 2250 7150 2700
@@
 	7300 3400 7150 3400
 Connection ~ 7150 3400
-$Comp
-L capacitive-pad:capacitive-pad C8
-U 1 1 5C6F4F8D
-P 7450 3850
-F 0 "C8" H 7677 3896 50  0000 L CNN
-F 1 "capacitive-pad" H 7677 3805 50  0000 L CNN
-F 2 "pads-cap-lib:capacitive-pad" H 7450 3850 50  0001 C CNN
-F 3 "" H 7450 3850 50  0001 C CNN
-	1    7450 3850
-	1    0    0    -1
-$EndComp
-Wire Wire Line
-	7150 3400 7150 3850
+Wire Wire Line
+	7150 3400 7150 3500
 Wire Wire Line
 	7150 3100 7050 3100
@@
 	7350 4600 7200 4600
 Connection ~ 7200 4600
-$Comp
-L capacitive-pad:capacitive-pad C10
-U 1 1 5C6F575B
-P 7500 5050
-F 0 "C10" H 7727 5096 50  0000 L CNN
-F 1 "capacitive-pad" H 7727 5005 50  0000 L CNN
-F 2 "pads-cap-lib:capacitive-pad" H 7500 5050 50  0001 C CNN
-F 3 "" H 7500 5050 50  0001 C CNN
-	1    7500 5050
-	1    0    0    -1
-$EndComp
 Wire Wire Line
 	7200 4600 7200 5050
@@
 	6450 2250 7150 2250
 Wire Wire Line
-	5400 3450 6700 3450
-Wire Wire Line
-	6700 3450 6700 3300
-Wire Wire Line
 	6700 3300 7050 3300
 Wire Wire Line
-	6800 3400 6800 3550
-Wire Wire Line
-	6800 3550 5400 3550
-Wire Wire Line
-	6800 3400 7150 3400
-Wire Wire Line
-	5400 3650 6800 3650
-Wire Wire Line
-	6800 3650 6800 4500
-Wire Wire Line
 	6800 4500 7100 4500
 Wire Wire Line
-	6700 4600 6700 3750
-Wire Wire Line
-	6700 3750 5400 3750
-Wire Wire Line
 	6700 4600 7200 4600
-NoConn ~ 5400 1350
-NoConn ~ 5400 1450
-NoConn ~ 5400 1550
 NoConn ~ 5400 2250
 NoConn ~ 5400 2350
-NoConn ~ 5400 2450
-NoConn ~ 5400 2550
 $Comp
 L Device:C C11
@@
 $EndComp
 Wire Wire Line
-	6450 3350 5400 3350
-Wire Wire Line
-	6450 2250 6450 3350
-Wire Wire Line
-	5400 3250 6350 3250
-Wire Wire Line
-	6350 3250 6350 2150
-Wire Wire Line
 	6050 3150 5400 3150
 Wire Wire Line
@@
 Wire Wire Line
 	6150 3050 6150 1150
+$Comp
+L capacitive-pad:capacitive-pad C4
+U 1 1 5C76C913
+P 7450 1600
+F 0 "C4" H 7677 1646 50  0000 L CNN
+F 1 "capacitive-pad" H 7677 1555 50  0000 L CNN
+F 2 "pads-cap-lib:capacitive-pad" H 7450 1600 50  0001 C CNN
+F 3 "" H 7450 1600 50  0001 C CNN
+	1    7450 1600
+	1    0    0    -1
+$EndComp
+$Comp
+L capacitive-pad:capacitive-pad C6
+U 1 1 5C76CB31
+P 7450 2700
+F 0 "C6" H 7677 2746 50  0000 L CNN
+F 1 "capacitive-pad" H 7677 2655 50  0000 L CNN
+F 2 "pads-cap-lib:capacitive-pad" H 7450 2700 50  0001 C CNN
+F 3 "" H 7450 2700 50  0001 C CNN
+	1    7450 2700
+	1    0    0    -1
+$EndComp
+$Comp
+L capacitive-pad:capacitive-pad C8
+U 1 1 5C76CBBD
+P 7450 3850
+F 0 "C8" H 7677 3896 50  0000 L CNN
+F 1 "capacitive-pad" H 7677 3805 50  0000 L CNN
+F 2 "pads-cap-lib:capacitive-pad" H 7450 3850 50  0001 C CNN
+F 3 "" H 7450 3850 50  0001 C CNN
+	1    7450 3850
+	1    0    0    -1
+$EndComp
+$Comp
+L capacitive-pad:capacitive-pad C10
+U 1 1 5C76CC31
+P 7500 5050
+F 0 "C10" H 7727 5096 50  0000 L CNN
+F 1 "capacitive-pad" H 7727 5005 50  0000 L CNN
+F 2 "pads-cap-lib:capacitive-pad" H 7500 5050 50  0001 C CNN
+F 3 "" H 7500 5050 50  0001 C CNN
+	1    7500 5050
+	1    0    0    -1
+$EndComp
+$Comp
+L MCU_Microchip_ATmega:ATmega168-20AU U1
+U 1 1 5C780DB7
+P 4800 2550
+F 0 "U1" H 4800 964 50  0000 C CNN
+F 1 "ATmega168-20AU" H 4800 873 50  0000 C CNN
+F 2 "Package_QFP:TQFP-32_7x7mm_P0.8mm" H 4800 2550 50  0001 C CIN
+F 3 "http://ww1.microchip.com/downloads/en/DeviceDoc/Atmel-2545-8-bit-AVR-Microcontroller-ATmega48-88-168_Datasheet.pdf" H 4800 2550 50  0001 C CNN
+	1    4800 2550
+	1    0    0    -1
+$EndComp
+NoConn ~ 4200 1550
+NoConn ~ 4200 1650
+Wire Wire Line
+	5400 2450 6350 2450
+Wire Wire Line
+	6350 2450 6350 2150
+Wire Wire Line
+	6450 2250 6450 2550
+Wire Wire Line
+	6450 2550 5400 2550
+$Comp
+L Device:R R6
+U 1 1 5C79139E
+P 7200 5600
+F 0 "R6" H 7270 5646 50  0000 L CNN
+F 1 "1M" H 7270 5555 50  0000 L CNN
+F 2 "Resistor_SMD:R_1206_3216Metric_Pad1.42x1.75mm_HandSolder" V 7130 5600 50  0001 C CNN
+F 3 "~" H 7200 5600 50  0001 C CNN
+	1    7200 5600
+	1    0    0    -1
+$EndComp
+$Comp
+L Device:C C12
+U 1 1 5C7913A5
+P 7500 5750
+F 0 "C12" V 7752 5750 50  0000 C CNN
+F 1 "100pF" V 7661 5750 50  0000 C CNN
+F 2 "Capacitor_SMD:C_1206_3216Metric_Pad1.42x1.75mm_HandSolder" H 7538 5600 50  0001 C CNN
+F 3 "~" H 7500 5750 50  0001 C CNN
+	1    7500 5750
+	0    -1   -1   0
+$EndComp
+$Comp
+L power:GND #PWR016
+U 1 1 5C7913AC
+P 7750 5750
+F 0 "#PWR016" H 7750 5500 50  0001 C CNN
+F 1 "GND" H 7755 5577 50  0000 C CNN
+F 2 "" H 7750 5750 50  0001 C CNN
+F 3 "" H 7750 5750 50  0001 C CNN
+	1    7750 5750
+	1    0    0    -1
+$EndComp
+Wire Wire Line
+	7750 5750 7650 5750
+Wire Wire Line
+	7350 5750 7200 5750
+Connection ~ 7200 5750
+Wire Wire Line
+	7200 5750 7200 6200
+Wire Wire Line
+	7200 5450 7100 5450
+Wire Wire Line
+	7100 5450 7100 5650
+$Comp
+L capacitive-pad:capacitive-pad C13
+U 1 1 5C7913BA
+P 7500 6200
+F 0 "C13" H 7727 6246 50  0000 L CNN
+F 1 "capacitive-pad" H 7727 6155 50  0000 L CNN
+F 2 "pads-cap-lib:capacitive-pad-small" H 7500 6200 50  0001 C CNN
+F 3 "" H 7500 6200 50  0001 C CNN
+	1    7500 6200
+	1    0    0    -1
+$EndComp
+Wire Wire Line
+	6250 5650 6250 1350
+Wire Wire Line
+	6250 1350 5400 1350
+Wire Wire Line
+	6250 5650 7100 5650
+Wire Wire Line
+	5400 3750 6150 3750
+Wire Wire Line
+	6150 3750 6150 5750
+Wire Wire Line
+	6150 5750 7200 5750
+NoConn ~ 5400 3250
+NoConn ~ 5400 1450
+NoConn ~ 5400 1550
+Wire Wire Line
+	5400 3550 6700 3550
+Wire Wire Line
+	6700 3550 6700 4600
+Wire Wire Line
+	6800 3650 5400 3650
+Wire Wire Line
+	6800 3650 6800 4500
+Wire Wire Line
+	5400 3450 6700 3450
+Wire Wire Line
+	6700 3300 6700 3450
+Wire Wire Line
+	5400 3350 7000 3350
+Wire Wire Line
+	7000 3350 7000 3500
+Wire Wire Line
+	7000 3500 7150 3500
+Connection ~ 7150 3500
+Wire Wire Line
+	7150 3500 7150 3850
 $EndSCHEMATC

Commit message: Fikset på kretskort
Parts:
- removed C12, C3, C5, C7, C9: 100pF, Capacitor_SMD:C_1206_3216Metric_Pad1.42x1.75mm_HandSolder, symbol Device:C
- J1: footprint Connector_PinHeader_1.27mm:PinHeader_1x05_P1.27mm_Vertical -> Connector_PinSocket_2.54mm:PinSocket_1x05_P2.54mm_Vertical_SMD_Pin1Left
- J2: footprint Connector_IDC:IDC-Header_2x03_P2.54mm_Vertical -> Connector_PinSocket_2.54mm:PinSocket_2x03_P2.54mm_Vertical_SMD
- Q1: footprint Package_TO_SOT_THT:TO-92L_Inline -> Package_TO_SOT_SMD:SOT-23_Handsoldering
Changed lines of the file:
@@
 F 0 "J1" H 2056 2528 50  0000 C CNN
 F 1 "Conn_01x05_Male" H 2056 2437 50  0000 C CNN
-F 2 "Connector_PinHeader_1.27mm:PinHeader_1x05_P1.27mm_Vertical" H 1950 2150 50  0001 C CNN
+F 2 "Connector_PinSocket_2.54mm:PinSocket_1x05_P2.54mm_Vertical_SMD_Pin1Left" H 1950 2150 50  0001 C CNN
 F 3 "~" H 1950 2150 50  0001 C CNN
 	1    1950 2150
@@
 	1    0    0    -1
 $EndComp
-$Comp
-L Device:C C3
-U 1 1 5C6F5DEA
-P 7450 1150
-F 0 "C3" V 7702 1150 50  0000 C CNN
-F 1 "100pF" V 7611 1150 50  0000 C CNN
-F 2 "Capacitor_SMD:C_1206_3216Metric_Pad1.42x1.75mm_HandSolder" H 7488 1000 50  0001 C CNN
-F 3 "~" H 7450 1150 50  0001 C CNN
-	1    7450 1150
-	0    -1   -1   0
-$EndComp
-$Comp
-L power:GND #PWR010
-U 1 1 5C6F5DF1
-P 7700 1150
-F 0 "#PWR010" H 7700 900 50  0001 C CNN
-F 1 "GND" H 7705 977 50  0000 C CNN
-F 2 "" H 7700 1150 50  0001 C CNN
-F 3 "" H 7700 1150 50  0001 C CNN
-	1    7700 1150
-	1    0    0    -1
-$EndComp
-Wire Wire Line
-	7700 1150 7600 1150
-Wire Wire Line
-	7300 1150 7150 1150
 Connection ~ 7150 1150
 NoConn ~ 4200 1350
@@
 F 0 "Q1" H 2955 2096 50  0000 L CNN
 F 1 "BS170" H 2955 2005 50  0000 L CNN
-F 2 "Package_TO_SOT_THT:TO-92L_Inline" H 2950 1975 50  0001 L CIN
+F 2 "Package_TO_SOT_SMD:SOT-23_Handsoldering" H 2950 1975 50  0001 L CIN
 F 3 "http://www.fairchildsemi.com/ds/BS/BS170.pdf" H 2750 2050 50  0001 L CNN
 	1    2750 2050
@@
 	1    0    0    -1
 $EndComp
-$Comp
-L Device:C C5
-U 1 1 5C6F49D6
-P 7450 2250
-F 0 "C5" V 7702 2250 50  0000 C CNN
-F 1 "100pF" V 7611 2250 50  0000 C CNN
-F 2 "Capacitor_SMD:C_1206_3216Metric_Pad1.42x1.75mm_HandSolder" H 7488 2100 50  0001 C CNN
-F 3 "~" H 7450 2250 50  0001 C CNN
-	1    7450 2250
-	0    -1   -1   0
-$EndComp
-$Comp
-L power:GND #PWR011
-U 1 1 5C6F49DD
-P 7700 2250
-F 0 "#PWR011" H 7700 2000 50  0001 C CNN
-F 1 "GND" H 7705 2077 50  0000 C CNN
-F 2 "" H 7700 2250 50  0001 C CNN
-F 3 "" H 7700 2250 50  0001 C CNN
-	1    7700 2250
-	1    0    0    -1
-$EndComp
-Wire Wire Line
-	7700 2250 7600 2250
-Wire Wire Line
-	7300 2250 7150 2250
 Connection ~ 7150 2250
 Wire Wire Line
@@
 	1    0    0    -1
 $EndComp
-$Comp
-L Device:C C7
-U 1 1 5C6F4F7D
-P 7450 3400
-F 0 "C7" V 7702 3400 50  0000 C CNN
-F 1 "100pF" V 7611 3400 50  0000 C CNN
-F 2 "Capacitor_SMD:C_1206_3216Metric_Pad1.42x1.75mm_HandSolder" H 7488 3250 50  0001 C CNN
-F 3 "~" H 7450 3400 50  0001 C CNN
-	1    7450 3400
-	0    -1   -1   0
-$EndComp
-$Comp
-L power:GND #PWR012
-U 1 1 5C6F4F84
-P 7700 3400
-F 0 "#PWR012" H 7700 3150 50  0001 C CNN
-F 1 "GND" H 7705 3227 50  0000 C CNN
-F 2 "" H 7700 3400 50  0001 C CNN
-F 3 "" H 7700 3400 50  0001 C CNN
-	1    7700 3400
-	1    0    0    -1
-$EndComp
-Wire Wire Line
-	7700 3400 7600 3400
-Wire Wire Line
-	7300 3400 7150 3400
-Connection ~ 7150 3400
 Wire Wire Line
 	7150 3400 7150 3500
@@
 	1    0    0    -1
 $EndComp
-$Comp
-L Device:C C9
-U 1 1 5C6F574B
-P 7500 4600
-F 0 "C9" V 7752 4600 50  0000 C CNN
-F 1 "100pF" V 7661 4600 50  0000 C CNN
-F 2 "Capacitor_SMD:C_1206_3216Metric_Pad1.42x1.75mm_HandSolder" H 7538 4450 50  0001 C CNN
-F 3 "~" H 7500 4600 50  0001 C CNN
-	1    7500 4600
-	0    -1   -1   0
-$EndComp
-$Comp
-L power:GND #PWR013
-U 1 1 5C6F5752
-P 7750 4600
-F 0 "#PWR013" H 7750 4350 50  0001 C CNN
-F 1 "GND" H 7755 4427 50  0000 C CNN
-F 2 "" H 7750 4600 50  0001 C CNN
-F 3 "" H 7750 4600 50  0001 C CNN
-	1    7750 4600
-	1    0    0    -1
-$EndComp
-Wire Wire Line
-	7750 4600 7650 4600
-Wire Wire Line
-	7350 4600 7200 4600
 Connection ~ 7200 4600
 Wire Wire Line
@@
 F 0 "J2" H 2120 4646 50  0000 R CNN
 F 1 "AVR-ISP-6" H 2120 4555 50  0000 R CNN
-F 2 "Connector_IDC:IDC-Header_2x03_P2.54mm_Vertical" V 2150 4600 50  0001 C CNN
+F 2 "Connector_PinSocket_2.54mm:PinSocket_2x03_P2.54mm_Vertical_SMD" V 2150 4600 50  0001 C CNN
 F 3 " ~" H 1125 4000 50  0001 C CNN
 	1    2400 4550
@@
 	1    0    0    -1
 $EndComp
-$Comp
-L Device:C C12
-U 1 1 5C7913A5
-P 7500 5750
-F 0 "C12" V 7752 5750 50  0000 C CNN
-F 1 "100pF" V 7661 5750 50  0000 C CNN
-F 2 "Capacitor_SMD:C_1206_3216Metric_Pad1.42x1.75mm_HandSolder" H 7538 5600 50  0001 C CNN
-F 3 "~" H 7500 5750 50  0001 C CNN
-	1    7500 5750
-	0    -1   -1   0
-$EndComp
-$Comp
-L power:GND #PWR016
-U 1 1 5C7913AC
-P 7750 5750
-F 0 "#PWR016" H 7750 5500 50  0001 C CNN
-F 1 "GND" H 7755 5577 50  0000 C CNN
-F 2 "" H 7750 5750 50  0001 C CNN
-F 3 "" H 7750 5750 50  0001 C CNN
-	1    7750 5750
-	1    0    0    -1
-$EndComp
-Wire Wire Line
-	7750 5750 7650 5750
-Wire Wire Line
-	7350 5750 7200 5750
 Connection ~ 7200 5750
 Wire Wire Line
